File: PowerOpAmps(TEC Drivers).sch (KiCad schematic (older format))
At the start: 0 parts

Commit message: added labels for loose ends
Parts:
- added C1: 100u, symbol Device:C
- added C3: 0.1u, symbol Device:C
- added R1: 470, symbol Device:R
- added U? (x2): OPA569AIDWPR, DWP20_4P32X3P81, symbol OPA569AIDWPR:OPA569AIDWPR
Connections:
- net labels added: GND, To_4.2V_Supply, To_Arduino_AtoD
- wire segments 0 -> 26
Changed lines of the file:
@@
 Comment4 ""
 $EndDescr
+$Comp
+L OPA569AIDWPR:OPA569AIDWPR U?
+U 1 1 60C92272
+P 3700 1800
+F 0 "U?" H 5600 2187 60  0000 C CNN
+F 1 "OPA569AIDWPR" H 5600 2081 60  0000 C CNN
+F 2 "DWP20_4P32X3P81" H 5600 2040 60  0001 C CNN
+F 3 "" H 3700 1800 60  0000 C CNN
+	1    3700 1800
+	1    0    0    -1
+$EndComp
+$Comp
+L OPA569AIDWPR:OPA569AIDWPR U?
+U 1 1 60C94364
+P 3750 4350
+F 0 "U?" H 5650 4737 60  0000 C CNN
+F 1 "OPA569AIDWPR" H 5650 4631 60  0000 C CNN
+F 2 "DWP20_4P32X3P81" H 5650 4590 60  0001 C CNN
+F 3 "" H 3750 4350 60  0000 C CNN
+	1    3750 4350
+	1    0    0    -1
+$EndComp
+Wire Wire Line
+	3700 1800 3600 1800
+Wire Wire Line
+	3450 1800 3450 1850
+Wire Wire Line
+	3700 2000 3600 2000
+Wire Wire Line
+	3600 2000 3600 1800
+Connection ~ 3600 1800
+Wire Wire Line
+	3600 1800 3450 1800
+$Comp
+L power:GND #PWR?
+U 1 1 60C996D8
+P 3450 1850
+F 0 "#PWR?" H 3450 1600 50  0001 C CNN
+F 1 "GND" H 3455 1677 50  0000 C CNN
+F 2 "" H 3450 1850 50  0001 C CNN
+F 3 "" H 3450 1850 50  0001 C CNN
+	1    3450 1850
+	1    0    0    -1
+$EndComp
+Wire Wire Line
+	8150 2200 8150 2100
+Connection ~ 8150 1900
+Connection ~ 8150 2100
+Wire Wire Line
+	8150 2100 8150 2000
+$Comp
+L power:GND #PWR?
+U 1 1 60C9A1CF
+P 8350 1950
+F 0 "#PWR?" H 8350 1700 50  0001 C CNN
+F 1 "GND" H 8355 1777 50  0000 C CNN
+F 2 "" H 8350 1950 50  0001 C CNN
+F 3 "" H 8350 1950 50  0001 C CNN
+	1    8350 1950
+	1    0    0    -1
+$EndComp
+Wire Wire Line
+	7500 2200 8150 2200
+Wire Wire Line
+	7500 2100 8150 2100
+Wire Wire Line
+	7500 1900 8150 1900
+Wire Wire Line
+	7500 2000 7650 2000
+Wire Wire Line
+	7650 2000 7650 1100
+Wire Wire Line
+	8150 1900 8350 1900
+Wire Wire Line
+	8350 1900 8350 1950
+Wire Wire Line
+	7650 2000 7750 2000
+Connection ~ 7650 2000
+Connection ~ 8150 2000
+Wire Wire Line
+	8150 2000 8150 1900
+$Comp
+L Device:R R1
+U 1 1 60C9D180
+P 7900 2000
+F 0 "R1" V 7693 2000 50  0000 C CNN
+F 1 "470" V 7784 2000 50  0000 C CNN
+F 2 "" V 7830 2000 50  0001 C CNN
+F 3 "~" H 7900 2000 50  0001 C CNN
+	1    7900 2000
+	0    1    1    0
+$EndComp
+Wire Wire Line
+	8050 2000 8150 2000
+Wire Wire Line
+	7500 2500 7500 2400
+Wire Wire Line
+	7500 2700 8000 2700
+Wire Wire Line
+	7500 2600 7600 2600
+Wire Wire Line
+	8000 2600 8000 2700
+Wire Wire Line
+	8000 2600 8250 2600
+Connection ~ 8000 2600
+$Comp
+L power:GND #PWR?
+U 1 1 60C9E215
+P 8000 3000
+F 0 "#PWR?" H 8000 2750 50  0001 C CNN
+F 1 "GND" H 8005 2827 50  0000 C CNN
+F 2 "" H 8000 3000 50  0001 C CNN
+F 3 "" H 8000 3000 50  0001 C CNN
+	1    8000 3000
+	1    0    0    -1
+$EndComp
+$Comp
+L power:GND #PWR?
+U 1 1 60C9E30F
+P 8250 2800
+F 0 "#PWR?" H 8250 2550 50  0001 C CNN
+F 1 "GND" H 8255 2627 50  0000 C CNN
+F 2 "" H 8250 2800 50  0001 C CNN
+F 3 "" H 8250 2800 50  0001 C CNN
+	1    8250 2800
+	1    0    0    -1
+$EndComp
+$Comp
+L Device:C C3
+U 1 1 60C9E72B
+P 8000 2850
+F 0 "C3" H 7750 2900 50  0000 L CNN
+F 1 "0.1u" H 7700 2800 50  0000 L CNN
+F 2 "" H 8038 2700 50  0001 C CNN
+F 3 "~" H 8000 2850 50  0001 C CNN
+	1    8000 2850
+	1    0    0    -1
+$EndComp
+Connection ~ 8000 2700
+$Comp
+L power:GND #PWR?
+U 1 1 60C9EDCF
+P 7500 2800
+F 0 "#PWR?" H 7500 2550 50  0001 C CNN
+F 1 "GND" H 7505 2627 50  0000 C CNN
+F 2 "" H 7500 2800 50  0001 C CNN
+F 3 "" H 7500 2800 50  0001 C CNN
+	1    7500 2800
+	1    0    0    -1
+$EndComp
+$Comp
+L Device:C C1
+U 1 1 60CA0405
+P 7750 2600
+F 0 "C1" V 7600 2500 50  0000 L CNN
+F 1 "100u" V 7600 2650 50  0000 L CNN
+F 2 "" H 7788 2450 50  0001 C CNN
+F 3 "~" H 7750 2600 50  0001 C CNN
+	1    7750 2600
+	0    1    1    0
+$EndComp
+Wire Wire Line
+	7900 2600 8000 2600
+Wire Wire Line
+	8250 2600 8250 2800
+Wire Wire Line
+	7500 2400 9050 2400
+Connection ~ 7500 2400
+Text Label 7400 1050 0    50   ~ 0
+To_Arduino_AtoD
+Text Label 9600 2700 0    50   ~ 0
+To_4.2V_Supply
+Wire Wire Line
+	8000 2700 9450 2700
 $EndSCHEMATC
