File: AtoD_DtoA.sch (KiCad schematic (older format))
At the start: 21 parts, among them IC701 ADS122C04IPWR, U701 MAX5217GUA+, U702 MAX5217GUA+

Commit message: name change on main for sheets
Parts:
- renumbered C709 to C?, C710 to C?, C711 to C?, C708 to C?, C707 to C?, C706 to C?, C705 to C?, C704 to C?, C703 to C?, C702 to C?, C701 to C?, IC701 to IC?, R707 to R?, R706 to R?, R705 to R?, R703 to R?, R704 to R?, R701 to R?, R702 to R?, U702 to U?, U701 to U?
