File: laser.sch (KiCad schematic (older format))
At the start: 1 part, among them U101 281698-3

Commit message: Finished.
Parts:
- added R101: 3.3k, Resistor_SMD:R_0402_1005Metric, symbol Device:R
Connections:
- net GND: now also R101.1
- net MODULATION_SIGNAL: now also R101.2
Changed lines of the file:
@@
 F1 "Butterfly.sch" 50
 $EndSheet
+$Comp
+L Device:R R101
+U 1 1 60EFE642
+P 10300 2550
+F 0 "R101" V 10093 2550 50  0000 C CNN
+F 1 "3.3k" V 10184 2550 50  0000 C CNN
+F 2 "Resistor_SMD:R_0402_1005Metric" V 10230 2550 50  0001 C CNN
+F 3 "~" H 10300 2550 50  0001 C CNN
+	1    10300 2550
+	0    1    1    0
+$EndComp
+Wire Wire Line
+	10450 2550 10650 2550
+$Comp
+L power:GND #PWR0111
+U 1 1 60EFF0B1
+P 10650 2550
+F 0 "#PWR0111" H 10650 2300 50  0001 C CNN
+F 1 "GND" H 10850 2500 50  0000 C CNN
+F 2 "" H 10650 2550 50  0001 C CNN
+F 3 "" H 10650 2550 50  0001 C CNN
+	1    10650 2550
+	1    0    0    -1
+$EndComp
+Wire Wire Line
+	10150 2550 9950 2550
+Wire Wire Line
+	9950 2550 9950 2800
 $EndSCHEMATC

Commit message: NEXT PROTO READY 8/5
Parts:
- R101: value 3.3k -> 100
Changed lines of the file:
@@
 P 10300 2550
 F 0 "R101" V 10093 2550 50  0000 C CNN
-F 1 "3.3k" V 10184 2550 50  0000 C CNN
+F 1 "100" V 10184 2550 50  0000 C CNN
 F 2 "Resistor_SMD:R_0402_1005Metric" V 10230 2550 50  0001 C CNN
 F 3 "~" H 10300 2550 50  0001 C CNN
